File: PCB_Power.kicad_sch (KiCad schematic)
At the start: 7 parts, among them J1 LiPo 3S, J2 Fligh Pin (Remove before flig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, J3 VOUT, Q1 2SJ555-E

Commit message: update
Parts:
- added Q2: 2SJ555-E, symbol Device:Q_PMOS_GDS
- J2: value Fligh Pin (Remove before flight tag) -> Remove before flight
Connections:
- net GND: now also C1.2, R1.2; no longer J2.2 (Pin_2)
- net at J3.1 (Pin_1): now also Q2.3 (S); no longer Q1.2 (D)
- net at J2.1 (Pin_1), Q1.1 (G): now also C1.1, R1.1, Q2.1 (G); no longer C1.2, R1.2
- net at F1.2, Q1.3 (S): now also J2.2 (Pin_2); no longer C1.1, R1.1
- new net: Q1.2 (D), Q2.2 (D)
Other:
- moved on the sheet: F1, J1, J3, Q1
